File: Elec Design/Slave Board/Slave Board.kicad_sch (KiCad schematic)
At the start: 77 parts, among them J1 JTAG, J2 OSTTC020162, J3 OSTTC030162, J4 OSTTC020162, J5 OSTTC030162, J6 0022232041, M1 VID28-05, M2 VID28-05, M3 VID28-05, M4 VID28-05, SW1 SW_SPST, U1 LPC11C22_24-LQFP48, U10 DRV5033AJxDBZ, U11 DRV5033AJxDBZ, U12 NCP718xSN500, U13 NCP718xSN330, U2 VID6606, U3 VID6606, U4 DRV5033AJxDBZ, U5 DRV5033AJxDBZ, U6 DRV5033AJxDBZ, U7 DRV5033AJxDBZ, U8 DRV5033AJxDBZ, U9 DRV5033AJxDBZ, Y1 12MHz/12pF

Commit message: converting to git structure
Parts:
- added C26: 10uF, Capacitor_SMD:C_0603_1608Metric, symbol Device:C
- added C27, C28: 0.1uF, Capacitor_SMD:C_0603_1608Metric, symbol Device:C
- added C29: 6800pF, Capacitor_SMD:C_0603_1608Metric, symbol Device:C
- added C30, C31: 22uF, Capacitor_SMD:C_0603_1608Metric, symbol Device:C
- added C32, C33: 1uF, Capacitor_SMD:C_0603_1608Metric, symbol Device:C
- added D5: B340, Diode_SMD:D_SMA, symbol Diode:B340
- added D6, D7: LED Low current, LED_SMD:LED_0603_1608Metric, symbol Device:LED
- added J8, J9: OSTTC020162, digikey-footprints:Term_Block_1x2_P5mm, symbol dk_Terminal-Blocks-Wire-to-Board:OSTTC020162
- added L1: 4.7uH, NR6028T4R7M:IND_NR6028T4R7M, symbol Device:L
- added R24: 10k, Resistor_SMD:R_0603_1608Metric, symbol Device:R
- added R25: 430k, Resistor_SMD:R_0603_1608Metric, symbol Device:R
- added R26: 82k, Resistor_SMD:R_0603_1608Metric, symbol Device:R
- added R27: 1k6, Resistor_SMD:R_0603_1608Metric, symbol Device:R
- added R28: 750R, Resistor_SMD:R_0603_1608Metric, symbol Device:R
- added R29, R30: 10k, Resistor_SMD:R_0805_2012Metric_Pad1.20x1.40mm_HandSolder, symbol Device:R
- added U14: BD9E302EFJ-E2, HTSOP-J8_ROM, symbol BD9E302EFJ-E2:BD9E302EFJ-E2
- added U15: NCP718xSN330, Package_TO_SOT_SMD:SOT-23-5, symbol Regulator_Linear:NCP718xSN330
Connections:
- net +3.3V: now also C33.1, R28.1, R29.1, R30.1, U15.5 (OUT)
- net +5V: now also C30.1, C31.1, C32.1, L1.2, R27.1, U15.1 (IN), U15.3 (EN)
- net CW/~{CCWB} - 1: now also R29.2
- net F(SCX)B - 1 : now also R30.2
- net GND: now also C26.2, C27.2, C30.2, C31.2, C32.2, C33.2, D6.1 (K), D7.1 (K), J8.2, J9.2, R24.2, R26.2, U14.4 (AGND), U14.7 (PGND), U14.EPAD, U15.2 (GND)
- net VBUS: now also D5.1 (K), J8.1, J9.1
- new net: C28.2, L1.1, R25.1, U14.8 (SW)
- new net: C26.1, C27.1, D5.2 (A), U14.2 (VIN), U14.3 (EN)
- new net: C29.1, U14.6 (COMP)
- new net: C29.2, R24.1
- new net: R25.2, R26.1, U14.5 (FB)
- new net: D6.2 (A), R27.2
- new net: D7.2 (A), R28.2
- new net: C28.1, U14.1 (BOOT)
Other:
- moved on the sheet: C14, C15, C17, C20, C25, D1, D2, D3, J2, J4, R14, R21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
