File: Elec Design/Main Board v1.4/Main Board.kicad_pcb (KiCad board)
At the start: 2 copper layers, 55.4 x 54.6 mm, 68 parts, among them J1 PJ-102A, J3 Conn_ARM_JTAG_SWD_10, J4 0022232041, SW1 SW_SPST, U1 BD9E302EFJ-E2, U2 ESP32-C3-MINI-1, U3 MCP2551-I-P, U4 NCP718xSN330, U5 LPC1768FBD100, Y1 12MHz/10pF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

Commit message: main board cleanup
Parts:
- moved C8 11.3 mm to (110.8, 118.0), turned to -90 degrees
- moved C10 10.2 mm to (112.5, 118.0), turned to -90 degrees
- moved R1 6.26 mm to (117.6, 110.5)
- moved L1 5.53 mm to (116.7, 115.6), turned to -90 degrees
- moved U4 4.01 mm to (108.1, 109.4), turned to 90 degrees
- moved R14 3.25 mm to (113.5, 105.5)
- moved D2 2.72 mm to (115.2, 104.5), turned to -90 degrees
- moved C12 2.10 mm to (109.0, 114.4), turned to -90 degrees
- moved R3 1.97 mm to (116.8, 106.0)
- moved C6 1.67 mm to (117.6, 108.8), turned to 180 degrees
- moved R4 0.48 mm to (118.5, 106.0), turned to -90 degrees
Connections:
- R3 pad 1: Net-(U1-SW) -> +5V
Routing:
- net GND: track 158.2 -> 151.4 mm, vias 29 -> 35
- net +5V: track 50.7 -> 56.9 mm, vias 1 -> 2
- net Net-(U1-SW): track 13.7 -> 9.36 mm
- net Net-(U3-TXD): track 8.26 -> 12.0 mm
- net Net-(U2-GPIO4/ADC1_CH4): track 29.9 -> 28.3 mm
- net Net-(U1-FB): track 5.62 -> 6.31 mm
- net Net-(C6-Pad2): track 2.30 -> 1.72 mm
- net Net-(U1-COMP): track 2.49 -> 3.02 mm
