File: Elec Design/Slave Board v1.3/Slave Board.kicad_pcb (KiCad board)
At the start: 2 copper layers, 81.3 x 358.6 mm, 101 parts, among them J3 1935174, J6 61300411121, J7 Conn_ARM_JTAG_SWD_10, J8 1935161, J9 1935161, M1 VID28-05, M2 VID28-05, M3 VID28-05, M4 VID28-05, SW1 SW_SPST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

Commit message: main board cleanup
Changed lines of the file:
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@@
 		(start 216.662 181.188)
 		(end 216.662 182.372)
-		(width 0.4064)
+		(width 0.5)
 		(layer "F.Cu")
 		(net 9)
@@
 		(start 217.25 177.55)
 		(end 217.25 180.6)
-		(width 0.4064)
+		(width 0.5)
 		(layer "F.Cu")
 		(net 9)
@@
 		(start 217.25 180.6)
 		(end 216.662 181.188)
-		(width 0.4064)
+		(width 0.5)
 		(layer "F.Cu")
 		(net 9)
